File: carte_pami/carte_pami.kicad_pcb (KiCad board)
At the start: 2 copper layers, 78 x 78 mm, 39 parts, among them J1 STEPPER, J2 STEPPER, J3 RANGE, J4 Screw_Terminal_01x02, J5 FDC, J6 FDC, J7 RANGE, J8 FDC, J9 UART, M1 Motor_Servo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

Commit message: routage by Fab
Parts:
- moved JP1 0.64 mm to (183.6, 79.4)
- moved JP2 0.64 mm to (183.6, 81.9)
- moved JP3 0.64 mm to (183.6, 84.5)
- moved R1 0.63 mm to (134.6, 31.8)
- moved JP5 0.25 mm to (183.0, 47.0)
- moved JP6 0.25 mm to (183.0, 44.5)
- moved JP4 0.25 mm to (183.0, 49.5)
Routing:
- net +3.3V: track 0.00 -> 184.4 mm, vias 0 -> 8
- net +5V: track 0.00 -> 120.7 mm
- net ALIM: track 0.00 -> 110.9 mm
- net STEP1_DIR: track 0.00 -> 78.2 mm, vias 0 -> 2
- net ENABLE: track 0.00 -> 69.5 mm, vias 0 -> 1
- net STEP1_PWM: track 0.00 -> 67.3 mm
- net STEP2_DIR: track 0.00 -> 38.5 mm
- net STEP2_PWM: track 0.00 -> 36.0 mm, vias 0 -> 2
- net MEAS_LIGHT: track 0.00 -> 29.3 mm
- net FDC1: track 0.00 -> 19.6 mm
- net SDA: track 0.00 -> 17.8 mm
- net SCL: track 0.00 -> 17.8 mm
- net SHUTDOWN1: track 0.00 -> 17.3 mm
- net FDC2: track 0.00 -> 16.4 mm
- net SHUTDOWN2: track 0.00 -> 15.5 mm, vias 0 -> 2
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- added copper zone on B.Cu, net GND
- added copper zone on F.Cu, net GND
