File: carte_pami/carte_pami.kicad_pcb (KiCad board)
At the start: 2 copper layers, 78 x 78 mm, 34 parts, among them J1 STEPPER, J2 STEPPER, J3 RANGE, J4 Screw_Terminal_01x02, J5 FDC2, J6 FDC1, J7 RANGE, J8 UART, M1 Motor_Servo, M2 Motor_Servo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

Commit message: Petits ajouts au schéma, et définition des capabilities.
Parts:
- added C5: 10uF, Capacitor_SMD:C_0805_2012Metric, F.Cu at (163.8, 80.3)
- added J9: UART, Connector_PinHeader_2.54mm:PinHeader_1x03_P2.54mm_Vertical, F.Cu at (163.2, 74.9)
- added M3: Motor_Servo, Connector_PinHeader_2.54mm:PinHeader_1x03_P2.54mm_Vertical, F.Cu at (131.4, 38.1)
- added R5: 2.2k, Resistor_SMD:R_0805_2012Metric, F.Cu at (151.5, 54.6)
- added R6: 2.2k, Resistor_SMD:R_0805_2012Metric, F.Cu at (151.5, 57.1)
- J5: value FDC2 -> FDC
- J6: value FDC1 -> FDC
- J8: value UART -> FDC; footprint Connector_PinHeader_2.54mm:PinHeader_1x04_P2.54mm_Vertical -> Connector_PinHeader_2.54mm:PinHeader_1x02_P2.54mm_Vertical
- moved J8 38.6 mm to (128.9, 59.7), turned to -90 degrees
- moved U2 22.2 mm to (168.9, 85.7)
- moved C4 16.2 mm to (167.6, 80.3)
- moved R3 16.0 mm to (128.9, 81.3)
- moved C3 15.7 mm to (170.2, 80.3)
- moved J5 12.1 mm to (128.9, 71.1)
- moved J6 10.8 mm to (128.9, 65.4)
- moved M1 6.63 mm to (131.4, 49.5)
- moved D1 4.97 mm to (126.5, 89.5), turned to 180 degrees
- moved M2 4.84 mm to (131.4, 43.8)
- moved R1 2.84 mm to (134.6, 32.4), turned to 0 degrees
- moved D2 2.38 mm to (134.5, 29.2)
- moved R2 2.34 mm to (130.5, 89.5), turned to 180 degrees
Connections:
- J8 pad 1: +5V -> FDC3
- U1 pad 19: unconnected-(U1-PA00-Pad19) -> SERVO3
- U1 pad 20: SERVO1 -> SERVO2
- U1 pad 21: SERVO2 -> SERVO1
- U1 pad 22: FDC2 -> FDC3
- U1 pad 23: FDC1 -> FDC2
- U1 pad 24: unconnected-(U1-PA06-Pad24) -> FDC1

Commit message: mesure batterie
Parts:
- removed J8: FDC, Connector_PinHeader_2.54mm:PinHeader_1x02_P2.54mm_Vertical
- added R7: 10k, Resistor_SMD:R_0805_2012Metric, F.Cu at (161.3, 80.4)
- added R8: 35k, Resistor_SMD:R_0805_2012Metric, F.Cu at (163.8, 80.4)
- moved R3 23.0 mm to (126.4, 58.4)
- moved C5 11.8 mm to (156.8, 89.8), turned to 90 degrees
- moved J6 1.91 mm to (128.9, 67.3)
- moved J5 1.91 mm to (128.9, 73.0)
Connections:
- U1 pad 22: FDC3 -> MEAS_LIGHT
- U1 pad 25: MEAS_LIGHT -> MEAS_BAT

Commit message: routage
Parts:
- moved J4 0.63 mm to (163.8, 99.1)
Routing:
- net +3.3V: track 0.00 -> 195.8 mm, vias 0 -> 5
- net ALIM: track 0.00 -> 115.2 mm, vias 0 -> 2
- net +5V: track 0.00 -> 99.3 mm, vias 0 -> 2
- net ENABLE: track 0.00 -> 74.7 mm, vias 0 -> 1
- net STEP1_DIR: track 0.00 -> 74.0 mm, vias 0 -> 2
- net STEP1_PWM: track 0.00 -> 64.4 mm
- net MEAS_BAT: track 0.00 -> 38.3 mm
- net STEP2_DIR: track 0.00 -> 35.7 mm
- net STEP2_PWM: track 0.00 -> 34.2 mm, vias 0 -> 2
- net FDC1: track 0.00 -> 22.2 mm
- net MEAS_LIGHT: track 0.00 -> 22.1 mm
- net GND: track 0.00 -> 21.0 mm, vias 0 -> 10
- net FDC2: track 0.00 -> 19.4 mm
- net SHUTDOWN1: track 0.00 -> 17.9 mm
- net SDA: track 0.00 -> 17.8 mm
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- added copper zone on B.Cu, net GND
Other:
- board text added: "SERVO 1"

Commit message: fini le routage de la carte
Parts:
- added G***: LOGO, ENAC_robotique:logo_enac_mini, F.Cu at (142.1, 96.2)
- added G***: LOGO, ENAC_robotique:logo_enac_mini, B.Cu at (142.7, 90.4)
- FDC 1: renamed from J5
- FDC 2: renamed from J6
- LED 1: renamed from D2
- LED 2: renamed from D1
- STEPPER 1: renamed from A1
- STEPPER 1: renamed from J1
- STEPPER 2: renamed from J2
- STEPPER 2: renamed from A2
- renumbered J4 to 12V, R3 to PHOTORESISTOR, J9 to UART
Other:
- board text added: "12V"
- board text added: "3.3V"
- board text added: "GND"
- board text added: "MAYSSEM & THOMAS @ ENAC 23"
- board text added: "MS1"
- board text added: "MS2"
- board text added: "MS3"
- board text added: "NUCLEO L432KC"
- board text added: "RX"
- board text added: "SCL"
- board text added: "SDA"
- board text added: "SERVO 2"
- board text added: "SERVO 3"
- board text added: "TX"
- board text added: "USB"
- board text added: "remove SB9 SB16 SB18"
