File: carte_pami/carte_pami.kicad_sch (KiCad schematic)
At the start: 39 parts, among them J1 STEPPER, J2 STEPPER, J3 RANGE, J4 Screw_Terminal_01x02, J5 FDC, J6 FDC, J7 RANGE, J8 FDC, J9 UART, M1 Motor_Servo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

Commit message: mesure batterie
Parts:
- removed J8: FDC, Connector_PinHeader_2.54mm:PinHeader_1x02_P2.54mm_Vertical, symbol Connector:Conn_01x02_Pin
- added R7: 10k, Resistor_SMD:R_0805_2012Metric, symbol Device:R_Small
- added R8: 35k, Resistor_SMD:R_0805_2012Metric, symbol Device:R_Small
Connections:
- net FDC3 is gone; now on net MEAS_LIGHT: U1.22 (PA04)
- net ALIM: now also R8.2
- net GND: now also R7.1
- net MEAS_LIGHT: no longer U1.25 (PA07)
- new net MEAS_BAT: R7.2, R8.1, U1.25 (PA07)
Other:
- note added: "Battery"
Changed lines of the file:
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@@
   (junction (at 242.57 96.52) (diameter 0) (color 0 0 0 0)
+  )
+  (junction (at 130.81 119.38) (diameter 0) (color 0 0 0 0)
   )
   (junction (at 86.36 48.26) (diameter 0) (color 0 0 0 0)
@@
     (stroke (width 0) (type default))
   )
+  (wire (pts (xy 132.08 119.38) (xy 130.81 119.38))
+    (stroke (width 0) (type default))
+  )
   (wire (pts (xy 222.25 127) (xy 227.33 127))
     (stroke (width 0) (type default))
   )
+  (wire (pts (xy 130.81 119.38) (xy 130.81 123.19))
+    (stroke (width 0) (type default))
+  )
   (wire (pts (xy 237.49 139.7) (xy 242.57 139.7))
     (stroke (width 0) (type default))
@@
     (stroke (width 0) (type default))
   )
+  (wire (pts (xy 130.81 130.81) (xy 130.81 128.27))
+    (stroke (width 0) (type default))
+  )
   (wire (pts (xy 247.65 96.52) (xy 242.57 96.52))
     (stroke (width 0) (type default))
   )
-  (wire (pts (xy 132.08 49.53) (xy 137.16 49.53))
-    (stroke (width 0) (type default))
-  )
   (wire (pts (xy 214.63 127) (xy 214.63 129.54))
     (stroke (width 0) (type default))
@@
     (stroke (width 0) (type default))
   )
+  (wire (pts (xy 130.81 114.3) (xy 130.81 119.38))
+    (stroke (width 0) (type default))
+  )
   (wire (pts (xy 227.33 109.22) (xy 227.33 111.76))
     (stroke (width 0) (type default))
@@
     (stroke (width 0) (type default))
   )
+  (wire (pts (xy 130.81 104.14) (xy 130.81 109.22))
+    (stroke (width 0) (type default))
+  )
   (wire (pts (xy 250.19 55.88) (xy 257.81 55.88))
     (stroke (width 0) (type default))
@@
   )
   (rectangle (start 205.74 19.05) (end 275.59 152.4)
+    (stroke (width 0) (type default))
+    (fill (type none))
+  )
+  (rectangle (start 125.73 90.17) (end 147.32 138.43)
     (stroke (width 0) (type default))
     (fill (type none))
@@
   )
   (text "Alim" (at 20.32 22.86 0)
+    (effects (font (size 2 2)) (justify left bottom))
+  )
+  (text "Battery" (at 127 93.98 0)
     (effects (font (size 2 2)) (justify left bottom))
   )
@@
     )
   )
-  (global_label "FDC3" (shape input) (at 132.08 46.99 0) (fields_autoplaced)
-    (effects (font (size 1.27 1.27)) (justify left))
-    (property "Intersheetrefs" "${INTERSHEET_REFS}" (at 139.9033 46.99 0)
-      (effects (font (size 1.27 1.27)) (justify left) hide)
-    )
-  )
   (global_label "STEP1_DIR" (shape input) (at 227.33 121.92 180) (fields_autoplaced)
     (effects (font (size 1.27 1.27)) (justify right))
@@
     )
   )
+  (global_label "ALIM" (shape input) (at 130.81 104.14 90) (fields_autoplaced)
+    (effects (font (size 1.27 1.27)) (justify left))
+    (property "Intersheetrefs" "${INTERSHEET_REFS}" (at 130.81 96.9819 90)
+      (effects (font (size 1.27 1.27)) (justify left) hide)
+    )
+  )
+  (global_label "MEAS_BAT" (shape input) (at 132.08 119.38 0) (fields_autoplaced)
+    (effects (font (size 1.27 1.27)) (justify left))
+    (property "Intersheetrefs" "${INTERSHEET_REFS}" (at 144.2575 119.38 0)
+      (effects (font (size 1.27 1.27)) (justify left) hide)
+    )
+  )
   (global_label "SERVO3" (shape input) (at 190.5 59.69 0) (fields_autoplaced)
     (effects (font (size 1.27 1.27)) (justify left))
@@
     )
   )
-  (global_label "FDC3" (shape input) (at 86.36 124.46 0) (fields_autoplaced)
-    (effects (font (size 1.27 1.27)) (justify left))
-    (property "Intersheetrefs" "${INTERSHEET_REFS}" (at 94.1833 124.46 0)
+  (global_label "MEAS_BAT" (shape input) (at 86.36 116.84 0) (fields_autoplaced)
+    (effects (font (size 1.27 1.27)) (justify left))
+    (property "Intersheetrefs" "${INTERSHEET_REFS}" (at 98.5375 116.84 0)
       (effects (font (size 1.27 1.27)) (justify left) hide)
     )
@@
     )
   )
-  (global_label "MEAS_LIGHT" (shape input) (at 86.36 116.84 0) (fields_autoplaced)
-    (effects (font (size 1.27 1.27)) (justify left))
-    (property "Intersheetrefs" "${INTERSHEET_REFS}" (at 100.4123 116.84 0)
+  (global_label "MEAS_LIGHT" (shape input) (at 86.36 124.46 0) (fields_autoplaced)
+    (effects (font (size 1.27 1.27)) (justify left))
+    (property "Intersheetrefs" "${INTERSHEET_REFS}" (at 100.4123 124.46 0)
       (effects (font (size 1.27 1.27)) (justify left) hide)
     )
@@
     )
   )
+  (symbol (lib_id "power:GND") (at 130.81 130.81 0) (unit 1)
+    (in_bom yes) (on_board yes) (dnp no) (fields_autoplaced)
+    (property "Reference" "#PWR034" (at 130.81 137.16 0)
+      (effects (font (size 1.27 1.27)) hide)
+    )
+    (property "Value" "GND" (at 130.81 135.89 0)
+      (effects (font (size 1.27 1.27)))
+    )
+    (property "Footprint" "" (at 130.81 130.81 0)
+      (effects (font (size 1.27 1.27)) hide)
+    )
+    (property "Datasheet" "" (at 130.81 130.81 0)
+      (effects (font (size 1.27 1.27)) hide)
+    )
+    (pin "1")
+    (instances
+      (project "carte_pami"
+        (path "/770e3594-3810-453e-8716-93c8c49f73f3"
+          (reference "#PWR034") (unit 1)
+        )
+      )
+    )
+  )
   (symbol (lib_id "power:+5V") (at 154.94 57.15 0) (unit 1)
     (in_bom yes) (on_board yes) (dnp no)
@@
     )
   )
-  (symbol (lib_id "Connector:Conn_01x02_Pin") (at 127 46.99 0) (unit 1)
-    (in_bom yes) (on_board yes) (dnp no)
-    (property "Reference" "J8" (at 124.46 49.53 0)
-      (effects (font (size 1.27 1.27)))
-    )
-    (property "Value" "FDC" (at 124.46 46.99 0)
-      (effects (font (size 1.27 1.27)))
-    )
-    (property "Footprint" "Connector_PinHeader_2.54mm:PinHeader_1x02_P2.54mm_Vertical" (at 127 46.99 0)
-      (effects (font (size 1.27 1.27)) hide)
-    )
-    (property "Datasheet" "~" (at 127 46.99 0)
-      (effects (font (size 1.27 1.27)) hide)
-    )
-    (pin "1")
-    (pin "2")
-    (instances
-      (project "carte_pami"
-        (path "/770e3594-3810-453e-8716-93c8c49f73f3"
-          (reference "J8") (unit 1)
-        )
-      )
-    )
-  )
   (symbol (lib_id "Connector:Conn_01x02_Pin") (at 125.73 36.83 0) (unit 1)
     (in_bom yes) (on_board yes) (dnp no)
@@
         (path "/770e3594-3810-453e-8716-93c8c49f73f3"
           (reference "#PWR02") (unit 1)
-        )
-      )
-    )
-  )
-  (symbol (lib_id "power:GND") (at 137.16 49.53 90) (unit 1)
-    (in_bom yes) (on_board yes) (dnp no) (fields_autoplaced)
-    (property "Reference" "#PWR034" (at 143.51 49.53 0)
-      (effects (font (size 1.27 1.27)) hide)
-    )
-    (property "Value" "GND" (at 140.97 49.53 90)
-      (effects (font (size 1.27 1.27)) (justify right))
-    )
-    (property "Footprint" "" (at 137.16 49.53 0)
-      (effects (font (size 1.27 1.27)) hide)
-    )
-    (property "Datasheet" "" (at 137.16 49.53 0)
-      (effects (font (size 1.27 1.27)) hide)
-    )
-    (pin "1")
-    (instances
-      (project "carte_pami"
-        (path "/770e3594-3810-453e-8716-93c8c49f73f3"
-          (reference "#PWR034") (unit 1)
         )
       )
@@
     )
   )
+  (symbol (lib_id "Device:R_Small") (at 130.81 111.76 180) (unit 1)
+    (in_bom yes) (on_board yes) (dnp no) (fields_autoplaced)
+    (property "Reference" "R8" (at 133.35 110.49 0)
+      (effects (font (size 1.27 1.27)) (justify right))
+    )
+    (property "Value" "35k" (at 133.35 113.03 0)
+      (effects (font (size 1.27 1.27)) (justify right))
+    )
+    (property "Footprint" "Resistor_SMD:R_0805_2012Metric" (at 130.81 111.76 0)
+      (effects (font (size 1.27 1.27)) hide)
+    )
+    (property "Datasheet" "~" (at 130.81 111.76 0)
+      (effects (font (size 1.27 1.27)) hide)
+    )
+    (pin "1")
+    (pin "2")
+    (instances
+      (project "carte_pami"
+        (path "/770e3594-3810-453e-8716-93c8c49f73f3"
+          (reference "R8") (unit 1)
+        )
+      )
+    )
+  )
   (symbol (lib_id "Device:C") (at 99.06 39.37 180) (unit 1)
     (in_bom yes) (on_board yes) (dnp no) (fields_autoplaced)
@@
         )
       )
+    )
+  )
+  (symbol (lib_id "Device:R_Small") (at 130.81 125.73 180) (unit 1)
+    (in_bom yes) (on_board yes) (dnp no) (fields_autoplaced)
+    (property "Reference" "R7" (at 133.35 124.46 0)
+      (effects (font (size 1.27 1.27)) (justify right))
+    )
+    (property "Value" "10k" (at 133.35 127 0)
+      (effects (font (size 1.27 1.27)) (justify right))
+    )
+    (property "Footprint" "Resistor_SMD:R_0805_2012Metric" (at 130.81 125.73 0)
+      (effects (font (size 1.27 1.27)) hide)
+    )
+    (property "Datasheet" "~" (at 130.81 125.73 0)
+      (effects (font (size 1.27 1.27)) hide)
+    )
+    (pin "1")
+    (pin "2")
+    (instances
+      (project "carte_pami"
+        (path "/770e3594-3810-453e-8716-93c8c49f73f3"
+          (reference "R7") (unit 1)
+        )
+      )
